File: devboard/nrf51822_devboard.rev2/nrf51822_devboard.kicad_pcb (KiCad board)
At the start: 4 copper layers, 50 x 50 mm, 34 parts, among them CON1 CORTEX-DEBUGGER, J1 microusb, J2 Conn_02x10_Odd_Even, J3 Conn_02x10_Odd_Even, SW1 SW_Push, SW2 SW_Push, U1 nRF51x22-QFxx, U2 LM1117-3.3, Y1 32.768, Y2 16MHz

Commit message: devboard
Other:
- board text added: "NRF51822"
